File: kicad-pcb/esp32-pedal-pcb.kicad_sch (KiCad schematic)
At the start: 40 parts, among them J1 USB_C_Receptacle_USB2.0_14P, Q1 Q_PMOS_GSD, U1 MCP73871, U2 TLV75733PDBV, U3 ESP32-S3-WROOM-1, U4 TPD2EUSB30, U5 TPD2E2U06DCK

Commit message: Update PCB design, documentation, and images
Parts:
- removed F1: Polyfuse_Small, Fuse:Fuse_Bourns_MF-RG500, symbol Device:Polyfuse_Small
- removed TP1: R+, TestPoint:TestPoint_Plated_Hole_D2.0mm, symbol Connector:TestPoint
- removed TP2: R-, TestPoint:TestPoint_Plated_Hole_D2.0mm, symbol Connector:TestPoint
- removed TP3, TP6: SW1, TestPoint:TestPoint_Plated_Hole_D2.0mm, symbol Connector:TestPoint
- removed TP4, TP7: SW GND, TestPoint:TestPoint_Plated_Hole_D2.0mm, symbol Connector:TestPoint
- removed TP5: SW2, TestPoint:TestPoint_Plated_Hole_D2.0mm, symbol Connector:TestPoint
- added R14: 100kΩ, Resistor_SMD:R_0603_1608Metric, symbol Device:R_US
- added TH1: Thermistor_NTC_US, Connector_Wire:SolderWire-0.5sqmm_1x02_P4.6mm_D0.9mm_OD2.1mm, symbol Device:Thermistor_NTC_US
- added TP1, TP2, TP3, TP4, TP5, TP6, TP7: TestPoint_Small, TestPoint_THTPad_D2.0mm_Drill1.0mm, symbol Connector:TestPoint_Small
- added U6: TPS2553DBVR, TPS2553DBVR:SOT95P280X145-6N, symbol Cossin:TPS2553DBVR
Connections:
- net GND: now also R14.2, TP4.1, TP7.1, U6.2 (GND)
- net VBUS: now also U6.1 (IN), U6.3 (EN)
- net VBUS PROTECTED: now also U6.6 (OUT); no longer R5.1
- net at U3.23 (GPIO21): now also TP6.1
- net at R5.2: now also C3.2, U1.1 (OUT), U1.20 (OUT); no longer U1.5 (THERM)
- net at U3.5 (GPIO5/TOUCH5/ADC1_CH4): now also TP3.1
- net at U3.7 (GPIO7/TOUCH7/ADC1_CH6): now also TP5.1
- net at C3.1: now also TP1.1; no longer U2.1 (IN)
- net BAT PROTECTED renamed VBAT
- net VBAT: no longer U2.3 (EN)
- new net: R14.1, U6.5 (ILIM)
- new net: R5.1, TH1.1
- new net: TH1.2, U1.5 (THERM)
- new net BAT SWITCHED: TP2.1, U2.1 (IN), U2.3 (EN)
- no-connect marks 29 -> 30
Other:
- moved on the sheet: R10, R11, R5
