File: kicad-pcb/esp32-pedal-pcb.kicad_sch (KiCad schematic)
At the start: 49 parts, among them J1 USB_C_Receptacle_USB2.0_14P, J2 Conn_01x03, J3 Conn_01x03, Q1 Q_PMOS_GSD, SW1 SW_SPST, SW2 SW_SPDT, U1 MCP73871, U2 TLV75733PDBV, U3 ESP32-S3-WROOM-1, U4 TPD2EUSB30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

Commit message: Update KiCad PCB project files and backups
Connections:
- net 3V3: now also R16.1, R17.1
- net Led DIN: now also U3.7 (GPIO7/TOUCH7/ADC1_CH6); no longer U3.38 (GPIO2/TOUCH2/ADC1_CH1)
- net at J2.3 (Pin_3), R19.2: now also U3.28 (SPIIO6/GPIO35/FSPID/SUBSPID); no longer U3.26 (GPIO45)
- net at J3.1 (Pin_1), R17.2: now also U3.38 (GPIO2/TOUCH2/ADC1_CH1); no longer U3.23 (GPIO21)
- net at J3.3 (Pin_3), R16.2: now also U3.29 (SPIIO7/GPIO36/FSPICLK/SUBSPICLK); no longer U3.16 (GPIO46)
- net at U3.39 (GPIO1/TOUCH1/ADC1_CH0): now also J2.1 (Pin_1), R18.2
- no-connect marks 28 -> 27
